Commit message: updated urdf file to match REP-105

File: ros_ws/src/greeter_description/urdf/robot.urdf (robot description, URDF)
Before this commit: robot theGreeter, 3 links, 2 joints
Links:
- removed link odom
- added link imu
Joints:
- removed joint odom_joint
- added joint imu_joint: type fixed, parent base_link, child imu_joint, origin xyz=0 0 0 rpy=0 0 0

Commit message: got odometry and IMU sensor data streaming

File: ros_ws/src/greeter_description/urdf/robot.urdf (robot description, URDF)
Before this commit: robot theGreeter, 3 links, 2 joints
Joints:
- joint imu_joint: child imu_joint -> imu
